File: PI_Shield.sch (EAGLE design)
At the start: 60 parts, among them Q1 220mA/50V/3.5Ω, Q3 220mA/50V/3.5Ω, Q4 220mA/50V/3.5Ω, U1 MAX1136EUA-T, U2 AZ1117EH-3.3TRG1, Y1 ECS-80-S-4X

Commit message: Update PI_Shield.sch
Parts:
- added D4: (no value), SparkFun-LED:LED0603
- added Q5: 2.5A/30V/105mΩ, SparkFun-DiscreteSemi:MOSFET_PCH-DMG2307L
- added R16: 1k, SparkFun-Resistors:RESISTOR0603
- added R17: 150, SparkFun-Resistors:RESISTOR0603
Connections:
- new net AMP_FAULT: Q5.G, R16.1
- new net N$10: Q5.S, R17.2
- new net N$11: D4.A, R17.1
- net 5V: now also Q5.D, R16.2
- net GND: now also D4.C
Other:
- note added: "LED on when Current Sensor Fault"
- note added: "PMOS"
Changed lines of the file:
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@@
 <part name="J7" library="SparkFun-Connectors" deviceset="CONN_02" device=""/>
 <part name="PCB1" library="MicrocontrollerComponents" deviceset="RPI2" device=""/>
+<part name="Q5" library="SparkFun-DiscreteSemi" library_urn="urn:adsk.eagle:library:514" deviceset="MOSFET_PCH" device="-DMG2307L" package3d_urn="urn:adsk.eagle:package:38446/1" value="2.5A/30V/105mΩ"/>
+<part name="R17" library="SparkFun-Resistors" library_urn="urn:adsk.eagle:library:532" deviceset="RESISTOR" device="0603" package3d_urn="urn:adsk.eagle:package:39650/1" value="150"/>
+<part name="D4" library="SparkFun-LED" library_urn="urn:adsk.eagle:library:529" deviceset="LED" device="0603" package3d_urn="urn:adsk.eagle:package:39354/1"/>
+<part name="R16" library="SparkFun-Resistors" library_urn="urn:adsk.eagle:library:532" deviceset="RESISTOR" device="0603" package3d_urn="urn:adsk.eagle:package:39650/1" value="1k"/>
 </parts>
 <sheets>
@@
 <text x="33.02" y="104.14" size="1.778" layer="91">Additional Analog Input Sensor</text>
 <text x="160.02" y="68.58" size="1.778" layer="91">3.3V Header Connectors</text>
+<text x="116.84" y="58.42" size="1.778" layer="91">PMOS</text>
+<text x="101.6" y="76.2" size="1.778" layer="91">LED on when Current Sensor Fault</text>
 </plain>
 <instances>
@@
 <attribute name="NAME" x="165.1" y="48.768" size="1.778" layer="95" font="vector"/>
 </instance>
+<instance part="Q5" gate="G$1" x="104.14" y="53.34" smashed="yes">
+<attribute name="NAME" x="109.22" y="53.34" size="1.778" layer="95" font="vector"/>
+<attribute name="VALUE" x="109.22" y="50.8" size="1.778" layer="96" font="vector"/>
+</instance>
+<instance part="R17" gate="G$1" x="114.3" y="40.64" smashed="yes" rot="R90">
+<attribute name="NAME" x="112.776" y="40.64" size="1.778" layer="95" font="vector" rot="R90" align="bottom-center"/>
+<attribute name="VALUE" x="115.824" y="40.64" size="1.778" layer="96" font="vector" rot="R90" align="top-center"/>
+</instance>
+<instance part="D4" gate="G$1" x="114.3" y="30.48" smashed="yes">
+<attribute name="NAME" x="110.871" y="25.908" size="1.778" layer="95" font="vector" rot="R90"/>
+<attribute name="VALUE" x="116.205" y="25.908" size="1.778" layer="96" font="vector" rot="R90" align="top-left"/>
+</instance>
+<instance part="R16" gate="G$1" x="93.98" y="60.96" smashed="yes" rot="R90">
+<attribute name="NAME" x="92.456" y="60.96" size="1.778" layer="95" font="vector" rot="R90" align="bottom-center"/>
+<attribute name="VALUE" x="95.504" y="60.96" size="1.778" layer="96" font="vector" rot="R90" align="top-center"/>
+</instance>
 </instances>
 <busses>
@@
 <wire x1="175.26" y1="43.18" x2="185.42" y2="43.18" width="0.1524" layer="91"/>
 <label x="180.34" y="43.18" size="1.778" layer="95"/>
+</segment>
+<segment>
+<pinref part="D4" gate="G$1" pin="C"/>
+<wire x1="114.3" y1="25.4" x2="114.3" y2="20.32" width="0.1524" layer="91"/>
+<label x="111.76" y="17.78" size="1.778" layer="95"/>
 </segment>
 </net>
@@
 <label x="66.04" y="129.54" size="1.778" layer="95"/>
 </segment>
+<segment>
+<pinref part="R16" gate="G$1" pin="2"/>
+<wire x1="93.98" y1="66.04" x2="93.98" y2="71.12" width="0.1524" layer="91"/>
+<label x="93.98" y="71.12" size="1.778" layer="95"/>
+</segment>
+<segment>
+<pinref part="Q5" gate="G$1" pin="D"/>
+<wire x1="106.68" y1="58.42" x2="106.68" y2="71.12" width="0.1524" layer="91"/>
+<label x="106.68" y="71.12" size="1.778" layer="95"/>
+</segment>
 </net>
 <net name="SDA" class="0">
@@
 </segment>
 </net>
+<net name="N$10" class="0">
+<segment>
+<pinref part="Q5" gate="G$1" pin="S"/>
+<wire x1="106.68" y1="48.26" x2="114.3" y2="48.26" width="0.1524" layer="91"/>
+<pinref part="R17" gate="G$1" pin="2"/>
+<wire x1="114.3" y1="48.26" x2="114.3" y2="45.72" width="0.1524" layer="91"/>
+</segment>
+</net>
+<net name="N$11" class="0">
+<segment>
+<pinref part="R17" gate="G$1" pin="1"/>
+<pinref part="D4" gate="G$1" pin="A"/>
+<wire x1="114.3" y1="35.56" x2="114.3" y2="33.02" width="0.1524" layer="91"/>
+</segment>
+</net>
+<net name="AMP_FAULT" class="0">
+<segment>
+<pinref part="Q5" gate="G$1" pin="G"/>
+<wire x1="99.06" y1="50.8" x2="93.98" y2="50.8" width="0.1524" layer="91"/>
+<pinref part="R16" gate="G$1" pin="1"/>
+<wire x1="93.98" y1="50.8" x2="93.98" y2="55.88" width="0.1524" layer="91"/>
+<wire x1="93.98" y1="50.8" x2="88.9" y2="50.8" width="0.1524" layer="91"/>
+<junction x="93.98" y="50.8"/>
+</segment>
+</net>
