File: PI_Shield.sch (EAGLE design)
At the start: 66 parts, among them Q1 220mA/50V/3.5Ω, Q3 220mA/50V/3.5Ω, Q4 220mA/50V/3.5Ω, Q5 2.5A/30V/105mΩ, U1 MAX1136EUA-T, U2 AZ1117EH-3.3TRG1, Y1 ECS-80-S-4X

Commit message: added note not to populate jumper
Other:
- note added: "Pull S pin high for silent mode Silent mode is unwanted Do not populate R3"
Changed lines of the file:
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@@
 <?xml version="1.0" encoding="utf-8"?>
 <!DOCTYPE eagle SYSTEM "eagle.dtd">
-<eagle version="8.6.1">
+<eagle version="9.1.3">
 <drawing>
 <settings>
@@
 <text x="213.36" y="88.9" size="1.778" layer="91">CAN to MiniROV Connectors</text>
 <text x="177.8" y="55.88" size="1.778" layer="91">NMOS</text>
+<text x="175.26" y="154.94" size="1.778" layer="91">Pull S pin high for silent mode
+Silent mode is unwanted
+Do not populate R3</text>
 </plain>
 <instances>

Commit message: Added comment
Added comment to not use two pins so that way board will not afect pi 4 boot-up
Other:
- note added: "DO NOT USE 27, 28"
- note added: "DO NOT use pin 28 or 27 these are form EEPROM"
- note added: "We will be using Pi 3, not Pi 2"
- note removed: "We will be using Pi 4, not Pi 2"
Changed lines of the file:
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@@
 <?xml version="1.0" encoding="utf-8"?>
 <!DOCTYPE eagle SYSTEM "eagle.dtd">
-<eagle version="9.1.3">
+<eagle version="9.6.2">
 <drawing>
 <settings>
@@
 <text x="5.08" y="35.56" size="1.778" layer="91">Data Logger Pin</text>
 <text x="43.18" y="33.02" size="1.778" layer="91">Data Logger Pin</text>
-<text x="71.12" y="63.5" size="1.778" layer="91" rot="R90">We will be using Pi 4, not Pi 2</text>
+<text x="71.12" y="63.5" size="1.778" layer="91" rot="R90">We will be using Pi 3, not Pi 2</text>
 <text x="134.62" y="27.94" size="1.778" layer="91">Sensors need to be assigned, chnage names later</text>
+<text x="45.72" y="121.92" size="1.778" layer="91" rot="R180">DO NOT use pin 28 or 27
+ these are form EEPROM</text>
+<text x="43.18" y="83.82" size="1.778" layer="91" rot="R180">DO NOT USE 27, 28</text>
 </plain>
 <instances>

Commit message: cad for 4 pin samtec t2i
Parts:
- removed U$13, U$14: T2I, BackplaneParts:T2I
- added U$15, U$5: T2I, Samtec t2i:T2I
Connections:
- net CANH: now also U$5.2; no longer U$13.2
- net CANL: now also U$5.3; no longer U$13.3
- net DI1: now also U$15.3; no longer U$14.3
- net DI2: now also U$15.2; no longer U$14.2
- net DI3: now also U$15.1; no longer U$14.1
- net GND: now also U$15.4; no longer U$14.4
Changed lines of the file:
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@@
 <part name="C6" library="SparkFun-Capacitors" library_urn="urn:adsk.eagle:library:510" deviceset="22NF/22,000PF" device="-0603-50V-10%" package3d_urn="urn:adsk.eagle:package:37414@1/1" value="4.7nF"/>
 <part name="U$10" library="BackplaneParts" deviceset="T2I" device=""/>
-<part name="U$13" library="BackplaneParts" deviceset="T2I" device=""/>
-<part name="U$14" library="BackplaneParts" deviceset="T2I" device=""/>
 <part name="R4" library="SparkFun-Resistors" library_urn="urn:adsk.eagle:library:532" deviceset="RESISTOR" device="0603" package3d_urn="urn:adsk.eagle:package:39650/1" value="470"/>
 <part name="R5" library="SparkFun-Resistors" library_urn="urn:adsk.eagle:library:532" deviceset="RESISTOR" device="0603" package3d_urn="urn:adsk.eagle:package:39650/1" value="68"/>
@@
 <part name="R18" library="SparkFun-Resistors" library_urn="urn:adsk.eagle:library:532" deviceset="RESISTOR" device="0603" package3d_urn="urn:adsk.eagle:package:39650/1" value="0"/>
 <part name="R21" library="SparkFun-Resistors" library_urn="urn:adsk.eagle:library:532" deviceset="RESISTOR" device="0603" package3d_urn="urn:adsk.eagle:package:39650/1" value="0"/>
+<part name="U$5" library="Samtec t2i" deviceset="T2I" device="" package3d_urn="urn:adsk.eagle:package:23194708/2"/>
+<part name="U$15" library="Samtec t2i" deviceset="T2I" device="" package3d_urn="urn:adsk.eagle:package:23194708/2"/>
 </parts>
 <sheets>
@@
 <attribute name="VALUE" x="228.6" y="144.78" size="1.778" layer="96" rot="R270"/>
 </instance>
-<instance part="U$13" gate="G$1" x="213.36" y="78.74" smashed="yes" rot="R270">
-<attribute name="NAME" x="220.98" y="86.36" size="1.778" layer="95" rot="R270"/>
-<attribute name="VALUE" x="215.9" y="86.36" size="1.778" layer="96" rot="R270"/>
-</instance>
-<instance part="U$14" gate="G$1" x="213.36" y="53.34" smashed="yes" rot="R270">
-<attribute name="NAME" x="220.98" y="60.96" size="1.778" layer="95" rot="R270"/>
-<attribute name="VALUE" x="215.9" y="60.96" size="1.778" layer="96" rot="R270"/>
-</instance>
 <instance part="R4" gate="G$1" x="160.02" y="58.42" smashed="yes" rot="R90">
 <attribute name="NAME" x="158.496" y="58.42" size="1.778" layer="95" font="vector" rot="R90" align="bottom-center"/>
@@
 <attribute name="NAME" x="55.88" y="37.084" size="1.778" layer="95" font="vector" align="bottom-center"/>
 <attribute name="VALUE" x="55.88" y="34.036" size="1.778" layer="96" font="vector" align="top-center"/>
+</instance>
+<instance part="U$5" gate="G$1" x="218.44" y="76.2" smashed="yes">
+<attribute name="NAME" x="215.9" y="78.74" size="1.778" layer="95"/>
+<attribute name="VALUE" x="215.9" y="63.5" size="1.778" layer="96"/>
+</instance>
+<instance part="U$15" gate="G$1" x="218.44" y="50.8" smashed="yes">
+<attribute name="NAME" x="215.9" y="53.34" size="1.778" layer="95"/>
+<attribute name="VALUE" x="215.9" y="38.1" size="1.778" layer="96"/>
 </instance>
 </instances>
@@
 </segment>
 <segment>
-<pinref part="U$14" gate="G$1" pin="4"/>
 <pinref part="GND11" gate="1" pin="GND"/>
 <wire x1="226.06" y1="43.18" x2="233.68" y2="43.18" width="0.1524" layer="91"/>
+<pinref part="U$15" gate="G$1" pin="4"/>
 </segment>
 <segment>
@@
 </segment>
 <segment>
-<pinref part="U$13" gate="G$1" pin="2"/>
 <wire x1="226.06" y1="73.66" x2="233.68" y2="73.66" width="0.1524" layer="91"/>
 <label x="228.6" y="73.66" size="1.778" layer="95"/>
+<pinref part="U$5" gate="G$1" pin="2"/>
 </segment>
 </net>
@@
 </segment>
 <segment>
-<pinref part="U$13" gate="G$1" pin="3"/>
 <wire x1="226.06" y1="71.12" x2="233.68" y2="71.12" width="0.1524" layer="91"/>
 <label x="228.6" y="71.12" size="1.778" layer="95"/>
+<pinref part="U$5" gate="G$1" pin="3"/>
 </segment>
 </net>
@@
 <net name="DI1" class="0">
 <segment>
-<pinref part="U$14" gate="G$1" pin="3"/>
 <wire x1="226.06" y1="45.72" x2="233.68" y2="45.72" width="0.1524" layer="91"/>
 <label x="231.14" y="45.72" size="1.778" layer="95"/>
+<pinref part="U$15" gate="G$1" pin="3"/>
 </segment>
 </net>
 <net name="DI2" class="0">
 <segment>
-<pinref part="U$14" gate="G$1" pin="2"/>
 <wire x1="226.06" y1="48.26" x2="233.68" y2="48.26" width="0.1524" layer="91"/>
 <label x="231.14" y="48.26" size="1.778" layer="95"/>
+<pinref part="U$15" gate="G$1" pin="2"/>
 </segment>
 </net>
 <net name="DI3" class="0">
 <segment>
-<pinref part="U$14" gate="G$1" pin="1"/>
 <wire x1="226.06" y1="50.8" x2="233.68" y2="50.8" width="0.1524" layer="91"/>
 <label x="231.14" y="50.8" size="1.778" layer="95"/>
-</segment>
-</net>
+<pinref part="U$15" gate="G$1" pin="1"/>
+</segment>
+</net>

Commit message: cad for 5 pin samtec t2i. had to reroute spi signals for larger t2i soldering area
Parts:
- removed U$8: T2I5P, BackplaneParts:T2I5P
- added U$13: T2I, Samtec t2i:T2I
- U$10: value T2I -> T2I5P; device BackplaneParts:T2I -> Samtec t2i:T2I5P
Connections:
- net 5V: now also U$10.1, U$10.2; no longer U$8.4, U$8.5
- net CANH: now also U$13.2; no longer U$10.2
- net CANL: now also U$13.3; no longer U$10.3
- net GND: now also U$10.4, U$10.5; no longer U$8.1, U$8.2
Changed lines of the file:
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@@
 <part name="R7" library="SparkFun-Resistors" library_urn="urn:adsk.eagle:library:532" deviceset="RESISTOR" device="0603" package3d_urn="urn:adsk.eagle:package:39650/1" value="60"/>
 <part name="C6" library="SparkFun-Capacitors" library_urn="urn:adsk.eagle:library:510" deviceset="22NF/22,000PF" device="-0603-50V-10%" package3d_urn="urn:adsk.eagle:package:37414@1/1" value="4.7nF"/>
-<part name="U$10" library="BackplaneParts" deviceset="T2I" device=""/>
 <part name="R4" library="SparkFun-Resistors" library_urn="urn:adsk.eagle:library:532" deviceset="RESISTOR" device="0603" package3d_urn="urn:adsk.eagle:package:39650/1" value="470"/>
 <part name="R5" library="SparkFun-Resistors" library_urn="urn:adsk.eagle:library:532" deviceset="RESISTOR" device="0603" package3d_urn="urn:adsk.eagle:package:39650/1" value="68"/>
@@
 <part name="R8" library="SparkFun-Resistors" library_urn="urn:adsk.eagle:library:532" deviceset="RESISTOR" device="0603" package3d_urn="urn:adsk.eagle:package:39650/1" value="330"/>
 <part name="R9" library="SparkFun-Resistors" library_urn="urn:adsk.eagle:library:532" deviceset="RESISTOR" device="0603" package3d_urn="urn:adsk.eagle:package:39650/1" value="330"/>
-<part name="U$8" library="BackplaneParts" deviceset="T2I5P" device=""/>
 <part name="J3" library="SparkFun-Connectors" library_urn="urn:adsk.eagle:library:513" deviceset="CONN_03" device="" package3d_urn="urn:adsk.eagle:package:38063/1"/>
 <part name="J5" library="SparkFun-Connectors" library_urn="urn:adsk.eagle:library:513" deviceset="CONN_02" device="" package3d_urn="urn:adsk.eagle:package:38039/1"/>
@@
 <part name="U$5" library="Samtec t2i" deviceset="T2I" device="" package3d_urn="urn:adsk.eagle:package:23194708/2"/>
 <part name="U$15" library="Samtec t2i" deviceset="T2I" device="" package3d_urn="urn:adsk.eagle:package:23194708/2"/>
+<part name="U$13" library="Samtec t2i" deviceset="T2I" device="" package3d_urn="urn:adsk.eagle:package:23194708/2"/>
+<part name="U$10" library="Samtec t2i" deviceset="T2I5P" device="" package3d_urn="urn:adsk.eagle:package:23194707/3"/>
 </parts>
 <sheets>
@@
 <attribute name="VALUE" x="204.724" y="122.301" size="1.778" layer="96" font="vector"/>
 </instance>
-<instance part="U$10" gate="G$1" x="226.06" y="137.16" smashed="yes" rot="R270">
-<attribute name="NAME" x="233.68" y="144.78" size="1.778" layer="95" rot="R270"/>
-<attribute name="VALUE" x="228.6" y="144.78" size="1.778" layer="96" rot="R270"/>
-</instance>
 <instance part="R4" gate="G$1" x="160.02" y="58.42" smashed="yes" rot="R90">
 <attribute name="NAME" x="158.496" y="58.42" size="1.778" layer="95" font="vector" rot="R90" align="bottom-center"/>
@@
 <attribute name="NAME" x="215.9" y="53.34" size="1.778" layer="95"/>
 <attribute name="VALUE" x="215.9" y="38.1" size="1.778" layer="96"/>
+</instance>
+<instance part="U$13" gate="G$1" x="231.14" y="134.62" smashed="yes">
+<attribute name="NAME" x="228.6" y="137.16" size="1.778" layer="95"/>
+<attribute name="VALUE" x="228.6" y="121.92" size="1.778" layer="96"/>
 </instance>
 </instances>
@@
 </segment>
 <segment>
-<pinref part="U$10" gate="G$1" pin="2"/>
 <wire x1="238.76" y1="132.08" x2="246.38" y2="132.08" width="0.1524" layer="91"/>
 <label x="241.3" y="132.08" size="1.778" layer="95"/>
+<pinref part="U$13" gate="G$1" pin="2"/>
 </segment>
 <segment>
@@
 </segment>
 <segment>
-<pinref part="U$10" gate="G$1" pin="3"/>
 <wire x1="238.76" y1="129.54" x2="246.38" y2="129.54" width="0.1524" layer="91"/>
 <label x="241.3" y="129.54" size="1.778" layer="95"/>
+<pinref part="U$13" gate="G$1" pin="3"/>
 </segment>
 <segment>
@@
 <attribute name="VALUE" x="193.04" y="130.556" size="1.778" layer="96" font="vector" align="top-center"/>
 </instance>
-<instance part="U$8" gate="&gt;NAME" x="182.88" y="93.98" smashed="yes" rot="R90">
-<attribute name="NAME" x="177.8" y="88.9" size="1.27" layer="95" rot="R90"/>
-</instance>
 <instance part="J3" gate="J$1" x="215.9" y="53.34" smashed="yes">
 <attribute name="VALUE" x="213.36" y="45.974" size="1.778" layer="96" font="vector"/>
@@
 <attribute name="NAME" x="241.3" y="102.616" size="1.778" layer="95" font="vector" rot="R180" align="bottom-center"/>
 <attribute name="VALUE" x="241.3" y="105.664" size="1.778" layer="96" font="vector" rot="R180" align="top-center"/>
+</instance>
+<instance part="U$10" gate="&gt;NAME" x="177.8" y="99.06" smashed="yes">
+<attribute name="NAME" x="182.88" y="101.6" size="1.27" layer="95" rot="MR0"/>
 </instance>
 </instances>
@@
 </segment>
 <segment>
-<pinref part="U$8" gate="&gt;NAME" pin="2"/>
 <wire x1="187.96" y1="91.44" x2="195.58" y2="91.44" width="0.1524" layer="91"/>
-<pinref part="U$8" gate="&gt;NAME" pin="1"/>
 <wire x1="187.96" y1="88.9" x2="195.58" y2="88.9" width="0.1524" layer="91"/>
 <wire x1="195.58" y1="91.44" x2="195.58" y2="88.9" width="0.1524" layer="91"/>
@@
 <wire x1="195.58" y1="88.9" x2="195.58" y2="86.36" width="0.1524" layer="91"/>
 <junction x="195.58" y="88.9"/>
+<pinref part="U$10" gate="&gt;NAME" pin="4"/>
+<pinref part="U$10" gate="&gt;NAME" pin="5"/>
 </segment>
 <segment>
@@
 </segment>
 <segment>
-<pinref part="U$8" gate="&gt;NAME" pin="4"/>
 <wire x1="187.96" y1="96.52" x2="195.58" y2="96.52" width="0.1524" layer="91"/>
-<pinref part="U$8" gate="&gt;NAME" pin="5"/>
-<wire x1="187.96" y1="99.06" x2="193.04" y2="99.06" width="0.1524" layer="91"/>
-<wire x1="193.04" y1="99.06" x2="195.58" y2="99.06" width="0.1524" layer="91"/>
+<wire x1="187.96" y1="99.06" x2="195.58" y2="99.06" width="0.1524" layer="91"/>
 <wire x1="195.58" y1="96.52" x2="195.58" y2="99.06" width="0.1524" layer="91"/>
 <pinref part="SUPPLY3" gate="G$1" pin="5V"/>
 <wire x1="195.58" y1="99.06" x2="195.58" y2="101.6" width="0.1524" layer="91"/>
 <junction x="195.58" y="99.06"/>
-</segment>
-<segment>
+<pinref part="U$10" gate="&gt;NAME" pin="1"/>
+<pinref part="U$10" gate="&gt;NAME" pin="2"/>
+</segment>
+<segment>
