File: PI_Shield.brd (EAGLE design)
At the start: 77.6 x 65.3 mm, 64 parts, among them Q1 220mA/50V/3.5Ω, Q3 220mA/50V/3.5Ω, Q4 220mA/50V/3.5Ω, Q5 2.5A/30V/105mΩ, U1 MAX1136EUA-T, U2 AZ1117EH-3.3TRG1, Y1 ECS-80-S-4X

Commit message: Update PI_Shield.brd
Parts:
- moved R7 1.43 mm to (53.5, 23.8)
- moved R20 1.27 mm to (85.1, 38.1)
- moved R3 1.04 mm to (53.2, 27.5)
- moved R2 0.95 mm to (64.1, 46.4)
Routing:
- net SCL: track 128.4 -> 120.1 mm
- net 3V3: track 282.5 -> 280.5 mm
- net MISO: track 35.0 -> 33.4 mm, vias 0 -> 1
- net DI: track 76.0 -> 74.5 mm, vias 3 -> 1
- net CANL: track 61.3 -> 62.7 mm
- net TXCAN: track 37.1 -> 35.6 mm
- net CS: track 32.8 -> 34.2 mm, vias 2 -> 3
- net N$6: track 7.58 -> 8.88 mm
- net N$9: track 16.0 -> 15.0 mm
- net N$1: track 5.89 -> 6.80 mm
- net SDA: track 108.7 -> 108.0 mm
- net CLK: track 33.8 -> 34.4 mm

Commit message: Update PI_Shield.brd
Routing:
- net IMU_RESET: track 41.4 -> 40.8 mm
Changed lines of the file:
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@@
 <wire x1="17.78" y1="28.545" x2="17.78" y2="29.5356" width="0.3048" layer="1"/>
 <wire x1="19.5118" y1="31.2674" x2="17.78" y2="29.5356" width="0.3048" layer="1"/>
-<wire x1="19.5118" y1="31.2674" x2="20.9804" y2="31.2674" width="0.3048" layer="1"/>
-<wire x1="20.9804" y1="31.2674" x2="28.6104875" y2="31.2674" width="0.3048" layer="1"/>
-<wire x1="18.385" y1="18.385" x2="17.78" y2="18.385" width="0.3048" layer="1"/>
-<wire x1="18.385" y1="18.385" x2="20.9804" y2="20.9804" width="0.3048" layer="1"/>
-<wire x1="45.72" y1="16.51" x2="40.64" y2="16.51" width="0.3048" layer="1"/>
-<wire x1="40.64" y1="26.67" x2="40.64" y2="16.51" width="0.3048" layer="1"/>
+<wire x1="19.5118" y1="31.2674" x2="20.447" y2="31.2674" width="0.3048" layer="1"/>
+<wire x1="20.447" y1="31.2674" x2="28.6104875" y2="31.2674" width="0.3048" layer="1"/>
+<wire x1="18.9184" y1="18.385" x2="17.78" y2="18.385" width="0.3048" layer="1"/>
+<wire x1="18.9184" y1="18.385" x2="20.447" y2="19.9136" width="0.3048" layer="1"/>
+<wire x1="45.72" y1="16.51" x2="41.5036" y2="16.51" width="0.3048" layer="1"/>
+<wire x1="41.5036" y1="27.5336" x2="41.5036" y2="16.51" width="0.3048" layer="1"/>
 <wire x1="88.9" y1="29.1592" x2="88.9" y2="25.4" width="0.3048" layer="1"/>
 <wire x1="87.63" y1="31.75" x2="81.28" y2="31.75" width="0.3048" layer="1"/>
@@
 <wire x1="40.0558" y1="39.37" x2="40.0558" y2="34.3662" width="0.254" layer="16"/>
 <wire x1="46.99" y1="51.22" x2="50.2" y2="51.22" width="0.3048" layer="1"/>
-<wire x1="40.64" y1="26.67" x2="41.5036" y2="27.5336" width="0.3048" layer="1"/>
 <wire x1="57.8866" y1="48.9204" x2="59.937" y2="46.87" width="0.3048" layer="1"/>
 <wire x1="59.937" y1="46.87" x2="60.96" y2="46.87" width="0.3048" layer="1"/>
@@
 <wire x1="44.45" y1="55.118" x2="45.2052" y2="55.8732" width="0.3048" layer="1"/>
 <wire x1="45.2052" y1="55.8732" x2="46.1332" y2="55.8732" width="0.3048" layer="1"/>
-<wire x1="20.9804" y1="20.9804" x2="20.9804" y2="31.2674" width="0.3048" layer="1"/>
+<wire x1="20.447" y1="19.9136" x2="20.447" y2="31.2674" width="0.3048" layer="1"/>
 <wire x1="65.532" y1="9.652" x2="67.31" y2="11.43" width="0.508" layer="16"/>
 <wire x1="55.88" y1="10.58" x2="57.9238" y2="10.58" width="0.508" layer="1"/>
-<wire x1="57.9238" y1="10.58" x2="58.4962" y2="10.0076" width="0.508" layer="1"/>
-<wire x1="58.4962" y1="10.0076" x2="65.8876" y2="10.0076" width="0.508" layer="1"/>
-<wire x1="65.8876" y1="10.0076" x2="67.31" y2="11.43" width="0.508" layer="1"/>
+<wire x1="57.9238" y1="10.58" x2="58.674" y2="9.8298" width="0.508" layer="1"/>
+<wire x1="58.674" y1="9.8298" x2="65.7098" y2="9.8298" width="0.508" layer="1"/>
+<wire x1="65.7098" y1="9.8298" x2="67.31" y2="11.43" width="0.508" layer="1"/>
 <wire x1="85.197" y1="43.0834" x2="83.6272" y2="44.6532" width="0.3048" layer="1"/>
 <wire x1="83.6272" y1="44.6532" x2="69.6468" y2="44.6532" width="0.3048" layer="1"/>
@@
 <wire x1="87.63" y1="31.75" x2="87.63" y2="30.4292" width="0.3048" layer="1"/>
 <wire x1="87.63" y1="30.4292" x2="88.9" y2="29.1592" width="0.3048" layer="1"/>
-<wire x1="35.83" y1="18.73" x2="35.83" y2="18.18289375" width="0.3048" layer="1"/>
-<wire x1="35.83" y1="18.18289375" x2="37.50289375" y2="16.51" width="0.3048" layer="1"/>
-<wire x1="37.50289375" y1="16.51" x2="40.64" y2="16.51" width="0.3048" layer="1"/>
+<wire x1="35.83" y1="18.73" x2="35.83" y2="18.23369375" width="0.3048" layer="1"/>
+<wire x1="35.83" y1="18.23369375" x2="37.55369375" y2="16.51" width="0.3048" layer="1"/>
+<wire x1="37.55369375" y1="16.51" x2="41.5036" y2="16.51" width="0.3048" layer="1"/>
 <via x="41.5036" y="27.5336" extent="1-16" drill="0.35"/>
 <via x="44.577" y="29.083" extent="1-16" drill="0.35"/>
@@
 <wire x1="31.75" y1="16.93" x2="31.85" y2="16.83" width="0.3048" layer="1"/>
 <wire x1="31.85" y1="16.83" x2="35.83" y2="16.83" width="0.3048" layer="1"/>
-<wire x1="27.5082" y1="19.7866" x2="27.5082" y2="19.4463125" width="0.3048" layer="1"/>
-<wire x1="27.5082" y1="19.4463125" x2="26.6038875" y2="18.542" width="0.3048" layer="1"/>
+<wire x1="27.5082" y1="19.7866" x2="27.5082" y2="19.4717125" width="0.3048" layer="1"/>
+<wire x1="27.5082" y1="19.4717125" x2="26.5784875" y2="18.542" width="0.3048" layer="1"/>
 <wire x1="21.3768" y1="18.542" x2="18.7198" y2="15.885" width="0.3048" layer="1"/>
 <wire x1="18.7198" y1="15.885" x2="17.78" y2="15.885" width="0.3048" layer="1"/>
-<wire x1="26.6038875" y1="18.542" x2="21.3768" y2="18.542" width="0.3048" layer="1"/>
+<wire x1="26.5784875" y1="18.542" x2="21.3768" y2="18.542" width="0.3048" layer="1"/>
 <wire x1="17.78" y1="26.045" x2="15.865" y2="26.045" width="0.3048" layer="1"/>
 <wire x1="15.865" y1="16.911" x2="15.865" y2="26.045" width="0.3048" layer="1"/>
@@
 <wire x1="57.8866" y1="17.8308" x2="56.2356" y2="19.4818" width="0.3048" layer="16"/>
 <wire x1="56.2356" y1="19.4818" x2="31.3182" y2="19.4818" width="0.3048" layer="16"/>
-<wire x1="28.9306" y1="21.8694" x2="28.9306" y2="29.4894" width="0.3048" layer="16"/>
+<wire x1="28.9306" y1="21.8694" x2="28.9306" y2="28.5242" width="0.3048" layer="16"/>
 <wire x1="31.3182" y1="19.4818" x2="28.9306" y2="21.8694" width="0.3048" layer="16"/>
-<wire x1="28.9306" y1="29.4894" x2="28.4734" y2="29.9466" width="0.3048" layer="16"/>
-<wire x1="28.4734" y1="29.9466" x2="27.5082" y2="29.9466" width="0.3048" layer="16"/>
+<wire x1="28.9306" y1="28.5242" x2="27.5082" y2="29.9466" width="0.3048" layer="16"/>
 </signal>
 <signal name="5V">
@@
 <contactref element="U$3" pad="INT"/>
 <contactref element="PCB1" pad="P$13"/>
-<wire x1="53.34" y1="34.29" x2="51.6382" y2="32.5882" width="0.3048" layer="16"/>
+<wire x1="53.34" y1="34.29" x2="53.34" y2="34.2392" width="0.3048" layer="16"/>
+<wire x1="53.34" y1="34.2392" x2="51.689" y2="32.5882" width="0.3048" layer="16"/>
 <wire x1="27.6098" y1="32.5882" x2="27.5082" y2="32.4866" width="0.3048" layer="16"/>
-<wire x1="51.6382" y1="32.5882" x2="27.6098" y2="32.5882" width="0.3048" layer="16"/>
+<wire x1="51.689" y1="32.5882" x2="27.6098" y2="32.5882" width="0.3048" layer="16"/>
 </signal>
 <signal name="DI">
@@
 <contactref element="PCB1" pad="P$2"/>
 <contactref element="PCB1" pad="P$4"/>
-<wire x1="24.9682" y1="19.7866" x2="24.9682" y2="17.2466" width="0.254" layer="16"/>
+<wire x1="24.9682" y1="17.2466" x2="24.9682" y2="19.7866" width="0.3048" layer="16"/>
 </signal>
 <signal name="AIN">

Commit message: Update PI_Shield.brd
Parts:
- moved R6 1.38 mm to (59.2, 19.9)
- moved C6 1.26 mm to (55.3, 19.9), turned to 270 degrees
- moved R8 0.20 mm to (52.3, 11.4)
Routing:
- net 3V3: track 280.4 -> 142.8 mm, vias 5 -> 3
- net 5V: track 143.8 -> 68.4 mm
- net PWM: track 63.1 -> 0.00 mm
- net AIN2: track 46.8 -> 0.00 mm, vias 2 -> 0
- net RXCAN: track 41.5 -> 0.00 mm, vias 5 -> 0
- net CANH: track 77.7 -> 39.8 mm, vias 1 -> 0
- net TXCAN: track 35.6 -> 0.00 mm, vias 7 -> 0
- net RESET_TO_PI: track 29.3 -> 0.00 mm, vias 1 -> 0
- net SDA: track 108.0 -> 82.6 mm
- net CANL: track 62.7 -> 43.2 mm, vias 1 -> 0
- net CS: track 34.2 -> 16.3 mm, vias 3 -> 0
- net SCL: track 120.1 -> 103.0 mm, vias 4 -> 3
- net FAULT: track 19.2 -> 2.79 mm, vias 2 -> 0
- net RESET: track 12.0 -> 0.00 mm, vias 2 -> 0
- net SCL_ADC: track 14.6 -> 4.33 mm
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
Commit message: Update PI_Shield.brd
Parts:
- moved J5 3.18 mm to (82.0, 58.8)
- moved R15 1.17 mm to (30.6, 31.6)
Routing:
- net 3V3: track 142.8 -> 248.0 mm, vias 3 -> 8
- net 5V: track 68.4 -> 138.8 mm, vias 0 -> 2
- net PWM: track 0.00 -> 64.8 mm
- net AIN2: track 0.00 -> 47.5 mm, vias 0 -> 2
- net RXCAN: track 0.00 -> 43.4 mm, vias 0 -> 3
- net TXCAN: track 0.00 -> 35.8 mm, vias 0 -> 3
- net CANH: track 39.8 -> 72.9 mm, vias 0 -> 1
- net RESET_TO_PI: track 0.00 -> 28.8 mm, vias 0 -> 3
- net SDA: track 82.6 -> 105.4 mm
- net SCL: track 103.0 -> 125.8 mm
- net CS: track 16.3 -> 37.4 mm, vias 0 -> 2
- net CANL: track 43.2 -> 60.6 mm
- net FAULT: track 2.79 -> 18.6 mm, vias 0 -> 2
- net RESET: track 0.00 -> 12.4 mm
- net SCL_ADC: track 4.33 -> 13.6 mm, vias 0 -> 2
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
Commit message: Update PI_Shield.brd
Routing:
- net 3V3: track 248.0 -> 246.2 mm
- net OSC1: track 6.92 -> 8.11 mm
Changed lines of the file:
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@@
 <contactref element="U$1" pad="OSC1"/>
 <contactref element="R19" pad="2"/>
-<wire x1="60.96" y1="62.23" x2="67.7046" y2="62.23" width="0.3048" layer="1"/>
 <wire x1="67.7046" y1="62.23" x2="67.8316" y2="62.103" width="0.3048" layer="1"/>
+<wire x1="60.96" y1="62.23" x2="62.9412" y2="62.23" width="0.3048" layer="1"/>
+<wire x1="62.9412" y1="62.23" x2="64.2874" y2="60.8838" width="0.3048" layer="1"/>
+<wire x1="64.2874" y1="60.8838" x2="65.7606" y2="60.8838" width="0.3048" layer="1"/>
+<wire x1="65.7606" y1="60.8838" x2="66.9798" y2="62.103" width="0.3048" layer="1"/>
+<wire x1="66.9798" y1="62.103" x2="67.8316" y2="62.103" width="0.3048" layer="1"/>
 </signal>
 <signal name="OSC2">
@@
 <wire x1="40.0796" y1="40.6654" x2="40.105" y2="40.64" width="0.3048" layer="1"/>
 <wire x1="37.0694" y1="40.6654" x2="40.0796" y2="40.6654" width="0.3048" layer="1"/>
-<wire x1="66.421" y1="23.0378" x2="68.1228" y2="23.0378" width="0.3048" layer="1"/>
-<wire x1="68.1228" y1="23.0378" x2="70.4088" y2="20.7518" width="0.3048" layer="1"/>
-<wire x1="70.4088" y1="20.7518" x2="73.3044" y2="20.7518" width="0.3048" layer="1"/>
-<wire x1="87.2236" y1="23.7236" x2="88.9" y2="25.4" width="0.3048" layer="1"/>
-<wire x1="73.3044" y1="20.7518" x2="76.2762" y2="23.7236" width="0.3048" layer="1"/>
-<wire x1="76.2762" y1="23.7236" x2="87.2236" y2="23.7236" width="0.3048" layer="1"/>
+<wire x1="68.7832" y1="23.4442" x2="68.3768" y2="23.0378" width="0.3048" layer="1"/>
+<wire x1="66.421" y1="23.0378" x2="68.3768" y2="23.0378" width="0.3048" layer="1"/>
+<wire x1="86.9442" y1="23.4442" x2="68.7832" y2="23.4442" width="0.3048" layer="1"/>
+<wire x1="86.9442" y1="23.4442" x2="88.9" y2="25.4" width="0.3048" layer="1"/>
 <wire x1="46.255" y1="40.64" x2="46.255" y2="49.3284" width="0.3048" layer="1"/>
 <wire x1="46.255" y1="49.3284" x2="46.99" y2="50.0634" width="0.3048" layer="1"/>
